File: Power Distribution.kicad_sch (KiCad schematic)
At the start: 16 parts, among them J1 Conn_01x02, J2 Conn_01x02, J3 Conn_01x02, J4 Conn_01x02, Q1 Q_PMOS_DGS

Commit message: Add files via upload
Changed some traces to adhere to new MOSFET footprint (from web library) and meet 0.3mm distance between all components. Addeed Gerber files.
Parts:
- Q1: footprint Transistor_Packages:SOT23_Standard -> DMP3056L-7 2:SOT91P240X110-3N
Changed lines of the file:
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@@
 			)
 		)
-		(property "Footprint" "Transistor_Packages:SOT23_Standard"
+		(property "Footprint" "DMP3056L-7 2:SOT91P240X110-3N"
 			(at 62.23 90.17 0)
 			(effects
